File: hardware/IoT_O2_Concentrator.kicad_sch (KiCad schematic)
At the start: 20 parts, among them J1 5V_BUCK_OUT, J10 12V_BUCK_IN, J11 O2_VCC_SEL, J12 BOX_SWITCH, J13 DC_MODULE, J2 BUZZER, J3 O2_SENSOR, J4 GPIOs, J5 RELAY, J6 LCD_20x04, J7 SIM_GSM_EVB, J8 POTENTIOMETER, J9 GPIO_SUPPLY

Commit message: Hardware v2.0: bare SIM800 module support and routing cleanup
Add JST for bare SIM module with 1N4001 drop from 5 V; remove O2 sensor voltage selector (sensor accepts 5 V). Replace routing jumpers with net ties (GND only) for DRC continuity; sheet version set to 2.0.
Parts:
- removed J11: O2_VCC_SEL, Connector_PinHeader_2.54mm:PinHeader_1x03_P2.54mm_Vertical, symbol Connector:Conn_01x03_Pin
- removed JP1: 5V_JUMPER, PCM_Jumper_AKL:Jumper_P7.62mm_D1.2mm, symbol Jumper:Jumper_2_Bridged
- removed JP2: GND_JUMPER, PCM_Jumper_AKL:Jumper_P7.62mm_D1.2mm, symbol Jumper:Jumper_2_Bridged
- removed JP3: 5V_JUMPER, PCM_Jumper_AKL:Jumper_P10.16mm_D1.2mm, symbol Jumper:Jumper_2_Bridged
- added D1: 1N4001, Diode_THT:D_DO-41_SOD81_P10.16mm_Horizontal, symbol Diode:1N4001
- added J14: SIM_GSM_BARE, footprint:JST_B5B-XH-A, symbol B5B-XH-A:B5B-XH-A
- added NT1: NetTie_2, PCM_SL_Jumpers:JUP_P10mm, symbol Device:NetTie_2
- J1: value 5V_BUCK_OUT -> 5V_LM2596
- J10: value 12V_BUCK_IN -> 12V_LM2596
Connections:
- net O2_VCC is gone; now on net 5V_VCC: J3.1
- net 5V_VCC: now also D1.2 (A)
- net GND: now also J14.5, NT1.1, NT1.2
- net SIM_RXD: now also J14.3
- net SIM_TXD: now also J14.4
- new net: D1.1 (K), J14.1
- no-connect marks 14 -> 15
Other:
- note added: "NC"
- moved on the sheet: A1, C1, C2, C3, J1, J10, J12, J13, J2, J3, J4, J5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
Changed lines of the file:
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@@
 	(title_block
 		(title "IoT_O2_Concentrator")
-		(date "2026-06-24")
-		(rev "1.0")
+		(date "2026-07-09")
+		(rev "2.0")
 		(company "---")
 	)

Commit message: Board V2 and firmware V2 implemented with softAP
Parts:
- added NT2: NetTie_2, PCM_SL_Jumpers:JUP_P10mm, symbol Device:NetTie_2
Connections:
- net GND: now also NT2.1, NT2.2
